File: IRseekerv2.kicad_sch (KiCad schematic)
At the start: 49 parts, among them J1 Conn_01x01_Pin, J13 Conn_01x04_Pin, J14 Conn_01x02_Pin, J16 G, J17 G, J18 G, J19 G, J20 Conn_01x02_Pin, J26 Conn_01x02_Pin, J27 Conn_01x02_Pin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

Commit message: STOP_COMM pin, solder pads for resistors on I2C lines
Parts:
- added J2: Conn_01x01_Pin, Connector_PinHeader_2.54mm:PinHeader_1x01_P2.54mm_Vertical, symbol Connector:Conn_01x01_Pin
- added JP1, JP2: SolderJumper_2_Open, Jumper:SolderJumper-2_P1.3mm_Open_TrianglePad1.0x1.5mm, symbol Jumper:SolderJumper_2_Open
Connections:
- net SCL: now also JP1.2 (B); no longer R4.2
- net SDA: now also JP2.1 (A); no longer R5.1
- net DISABLE_COMM: now reaches U3.32 (PA10)
- net DISABLE_COMM: now also J2.1 (Pin_1)
- new net: JP2.2 (B), R5.1
- new net: JP1.1 (A), R4.2
Other:
- moved on the sheet: J26, R4, R5
